File: pcbs/curcur40/pmw3360/curcur40-pmw3360.kicad_sch (KiCad schematic)
At the start: 20 parts, among them J1 Conn_01x08, U1 PMW3360, U2 TLV74318PDBVR

Commit message: fix
Parts:
- H1, H2, H3, H4: value MountingHole_Pad -> MountingHole_2.2mm_M2; footprint MountingHole:MountingHole_3.2mm_M3_ISO14580 -> MountingHole:MountingHole_2.2mm_M2
Changed lines of the file:
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@@
 			)
 		)
-		(property "Value" "MountingHole_Pad"
+		(property "Value" "MountingHole_2.2mm_M2"
 			(at 237.49 128.2699 0)
 			(hide yes)
@@
 			)
 		)
-		(property "Footprint" "MountingHole:MountingHole_3.2mm_M3_ISO14580"
+		(property "Footprint" "MountingHole:MountingHole_2.2mm_M2"
 			(at 234.95 128.27 0)
 			(hide yes)
@@
 			)
 		)
-		(property "Value" "MountingHole_Pad"
+		(property "Value" "MountingHole_2.2mm_M2"
 			(at 242.57 128.2699 0)
 			(hide yes)
@@
 			)
 		)
-		(property "Footprint" "MountingHole:MountingHole_3.2mm_M3_ISO14580"
+		(property "Footprint" "MountingHole:MountingHole_2.2mm_M2"
 			(at 240.03 128.27 0)
 			(hide yes)
@@
 			)
 		)
-		(property "Value" "MountingHole_Pad"
+		(property "Value" "MountingHole_2.2mm_M2"
 			(at 232.41 128.2699 0)
 			(hide yes)
@@
 			)
 		)
-		(property "Footprint" "MountingHole:MountingHole_3.2mm_M3_ISO14580"
+		(property "Footprint" "MountingHole:MountingHole_2.2mm_M2"
 			(at 229.87 128.27 0)
 			(hide yes)
@@
 			)
 		)
-		(property "Value" "MountingHole_Pad"
+		(property "Value" "MountingHole_2.2mm_M2"
 			(at 247.65 128.2699 0)
 			(hide yes)
@@
 			)
 		)
-		(property "Footprint" "MountingHole:MountingHole_3.2mm_M3_ISO14580"
+		(property "Footprint" "MountingHole:MountingHole_2.2mm_M2"
 			(at 245.11 128.27 0)
 			(hide yes)
