File: pcbs/curcur40/right/curcur40-right.kicad_pcb (KiCad board)
At the start: 2 copper layers, 124.3 x 91.8 mm, 81 parts

Commit message: fix all
Parts:
- moved rH1 2.00 mm to (5.03, 42.4)
- moved rH3 2.00 mm to (5.03, 62.4)
- moved rH2 2.00 mm to (14.0, 42.4)
- moved rH4 2.00 mm to (14.0, 62.4)
Routing:
- net /SCLK: track 119.9 -> 122.6 mm
- net /MOSI: track 119.1 -> 121.3 mm
- net /MISO: track 123.0 -> 124.7 mm
Other:
- outline, holes or cut-outs redrawn
Changed lines of the file:
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@@
 	(footprint ""
 		(layer "F.Cu")
-		(at 12.025 62.3875)
+		(at 14.025 62.3875)
 		(property "Reference" "rH4"
 			(at 0 0 0)
@@
 	(footprint ""
 		(layer "F.Cu")
-		(at 12.025 42.3875)
+		(at 14.025 42.3875)
 		(property "Reference" "rH2"
 			(at 0 0 0)
@@
 	(footprint ""
 		(layer "F.Cu")
-		(at 3.025 42.3875)
+		(at 5.025 42.3875)
 		(property "Reference" "rH1"
 			(at 0 0 0)
@@
 	(footprint ""
 		(layer "F.Cu")
-		(at 3.025 62.3875)
+		(at 5.025 62.3875)
 		(property "Reference" "rH3"
 			(at 0 0 0)
@@
 	(gr_line
 		(start -4.263 67.5)
-		(end 18.5 67.5)
+		(end 20.5 67.5)
 		(stroke
 			(width 0.15)
@@
 		(layer "Edge.Cuts")
 	)
-	(gr_circle
-		(center 7.525 52.3875)
-		(end 12.525 52.3875)
-		(stroke
-			(width 0.15)
-			(type default)
-		)
-		(fill no)
-		(layer "Edge.Cuts")
-	)
 	(gr_line
 		(start 7.667502 -17.16875)
@@
 		(layer "Edge.Cuts")
 	)
+	(gr_circle
+		(center 9.525 52.3875)
+		(end 14.525 52.3875)
+		(stroke
+			(width 0.15)
+			(type default)
+		)
+		(fill no)
+		(layer "Edge.Cuts")
+	)
 	(gr_line
 		(start 16.907502 -17.16875)
@@
 	)
 	(gr_line
-		(start 18.5 67.5)
-		(end 22.8375 63.1625)
-		(stroke
-			(width 0.15)
-			(type default)
-		)
-		(layer "Edge.Cuts")
-	)
-	(gr_line
-		(start 22.8375 63.1625)
-		(end 81.463 63.1625)
+		(start 20.5 67.5)
+		(end 24.8375 63.1625)
 		(stroke
 			(width 0.15)
@@
 	)
 	(gr_line
+		(start 24.8375 63.1625)
+		(end 81.463 63.1625)
+		(stroke
+			(width 0.15)
+			(type default)
+		)
+		(layer "Edge.Cuts")
+	)
+	(gr_line
 		(start 42.362504 -19.55)
 		(end 42.362504 -20.93125)
@@
 	)
 	(segment
+		(start 20 60.712)
+		(end 16.512 64.2)
+		(width 0.2)
+		(layer "B.Cu")
+		(net "+3V3R")
+	)
+	(segment
 		(start 64.6175 34.27625)
 		(end 70.433752 34.27625)
@@
 	)
 	(segment
+		(start 16.512 64.2)
+		(end 1.2 64.2)
+		(width 0.2)
+		(layer "B.Cu")
+		(net "+3V3R")
+	)
+	(segment
 		(start 58.8175 10.30625)
 		(end 58.9075 10.21625)
@@
 	)
 	(segment
-		(start 14.512 64.2)
-		(end 1.2 64.2)
-		(width 0.2)
-		(layer "B.Cu")
-		(net "+3V3R")
-	)
-	(segment
 		(start 64.3575 34.01625)
 		(end 63.8275 34.01625)
@@
 	)
 	(segment
+		(start 1.2 64.2)
+		(end 1.2 60.712)
+		(width 0.2)
+		(layer "B.Cu")
+		(net "+3V3R")
+	)
+	(segment
 		(start 63.8275 31.91625)
 		(end 63.8275 34.01625)
@@
 	)
 	(segment
+		(start 63.8 60.712)
+		(end 20 60.712)
+		(width 0.2)
+		(layer "B.Cu")
+		(net "+3V3R")
+	)
+	(segment
 		(start 85.592508 37.75875)
 		(end 85.632508 37.79875)
@@
 	)
 	(segment
-		(start 18 60.712)
-		(end 14.512 64.2)
-		(width 0.2)
-		(layer "B.Cu")
-		(net "+3V3R")
-	)
-	(segment
-		(start 63.8 60.712)
-		(end 18 60.712)
-		(width 0.2)
-		(layer "B.Cu")
-		(net "+3V3R")
-	)
-	(segment
 		(start 74.4075 41.0774)
 		(end 74.4075 42.2425)
@@
 	)
 	(segment
-		(start 1.2 64.2)
-		(end 1.2 60.712)
-		(width 0.2)
-		(layer "B.Cu")
-		(net "+3V3R")
-	)
-	(segment
 		(start 68.6075 31.61625)
 		(end 68.2025 31.61625)
@@
 	)
 	(segment
-		(start 19.799999 62.362)
-		(end 16.161999 66)
+		(start 21.799999 62.362)
+		(end 18.162 66)
 		(width 0.2)
 		(layer "B.Cu")
@@
 	)
 	(segment
-		(start 79.6 62.362)
-		(end 19.799999 62.362)
+		(start 77.42 38.22)
+		(end 77.3 38.1)
 		(width 0.2)
 		(layer "B.Cu")
@@
 	)
 	(segment
-		(start 16.161999 66)
-		(end -1 66)
+		(start -1 66)
+		(end -1 54.151)
 		(width 0.2)
 		(layer "B.Cu")
@@
 	)
 	(segment
-		(start 77.42 38.22)
-		(end 77.3 38.1)
+		(start 18.162 66)
+		(end -1 66)
 		(width 0.2)
 		(layer "B.Cu")
@@
 	)
 	(segment
-		(start -1 66)
-		(end -1 54.151)
+		(start 79.6 62.362)
+		(end 21.799999 62.362)
+		(width 0.2)
+		(layer "B.Cu")
+		(net "/MISO")
+	)
+	(segment
+		(start -1 54.151)
+		(end -2.725 54.151)
 		(width 0.2)
 		(layer "B.Cu")
@@
 	)
 	(segment
-		(start 15.611999 65.4)
-		(end -0.5 65.4)
+		(start 78.95 61.812)
+		(end 21.2 61.812)
 		(width 0.2)
 		(layer "B.Cu")
@@
 	)
 	(segment
-		(start 78.95 61.812)
-		(end 19.2 61.812)
+		(start 21.2 61.812)
+		(end 17.611999 65.4)
 		(width 0.2)
 		(layer "B.Cu")
@@
 	)
 	(segment
-		(start 19.2 61.812)
-		(end 15.611999 65.4)
+		(start -0.5 65.4)
+		(end -0.5 51.611)
 		(width 0.2)
 		(layer "B.Cu")
@@
 	)
 	(segment
-		(start -0.5 65.4)
-		(end -0.5 51.611)
+		(start -0.5 51.611)
+		(end -2.725 51.611)
 		(width 0.2)
 		(layer "B.Cu")
@@
 	)
 	(segment
+		(start 17.611999 65.4)
+		(end -0.5 65.4)
+		(width 0.2)
+		(layer "B.Cu")
+		(net "/MOSI")
+	)
+	(segment
 		(start 78.045 40.8)
 		(end 78.95 41.705)
@@
 	)
 	(segment
-		(start 18.599999 61.263)
-		(end 15.062999 64.8)
-		(width 0.2)
-		(layer "B.Cu")
-		(net "/SCLK")
-	)
-	(segment
 		(start 78.3 61.263)
-		(end 18.599999 61.263)
+		(end 20.599999 61.263)
 		(width 0.2)
 		(layer "B.Cu")
@@
 	)
 	(segment
+		(start 20.599999 61.263)
+		(end 17.062999 64.8)
+		(width 0.2)
+		(layer "B.Cu")
+		(net "/SCLK")
+	)
+	(segment
 		(start 76.7625 41.953)
 		(end 77.9 41.953)
@@
 	)
 	(segment
-		(start 15.062999 64.8)
+		(start 0 49.071)
+		(end -2.725 49.071)
+		(width 0.2)
+		(layer "B.Cu")
+		(net "/SCLK")
+	)
+	(segment
+		(start 17.062999 64.8)
 		(end 0 64.8)
 		(width 0.2)
@@
 	)
 	(segment
-		(start 23.575 42.416)
-		(end 15.5 42.416)
-		(width 0.2)
-		(layer "B.Cu")
-		(net "/TX")
-	)
-	(segment
-		(start 11.63 38.546)
-		(end 10.268 38.546)
-		(width 0.2)
-		(layer "B.Cu")
-		(net "/TX")
-	)
-	(segment
 		(start 40.9675 40.50125)
 		(end 40.6684 40.80035)
@@
 	)
 	(segment
-		(start 15.5 42.416)
-		(end 11.63 38.546)
+		(start 13.63 38.546)
+		(end 10.268 38.546)
+		(width 0.2)
+		(layer "B.Cu")
+		(net "/TX")
+	)
+	(segment
+		(start 17.5 42.416)
+		(end 13.63 38.546)
 		(width 0.2)
 		(layer "B.Cu")
@@
 		(layer "B.Cu")
 		(net "/TX")
+	)
+	(segment
+		(start 23.575 42.416)
+		(end 17.5 42.416)
+		(width 0.2)
+		(layer "B.Cu")
+		(net "/TX")

Commit message: fix all
Parts:
- moved rJ2 9.53 mm to (-5.26, 34.6)
- moved rJ1 7.09 mm to (12.3, -23.1)
Routing:
- net +5VR: track 107.4 -> 138.5 mm
- net /D+: track 128.3 -> 142.5 mm
- net VBUSR: track 15.0 -> 29.2 mm
- net /D-: track 133.3 -> 147.5 mm
- net /TX: track 95.0 -> 106.5 mm, vias 2 -> 3
- net Net-(rJ1-CC1): track 11.5 -> 18.6 mm
- net Net-(rJ1-CC2): track 11.1 -> 18.2 mm
Other:
- outline, holes or cut-outs redrawn

Commit message: Restore TRRS cutouts and relocate mounting holes to perimeter
Routing:
- net /NCS: track 154.3 -> 170.5 mm
- net +5VR: track 138.5 -> 123.1 mm
- net GNDR: track 142.8 -> 145.0 mm
- net /TX: track 106.5 -> 108.6 mm
Other:
- outline, holes or cut-outs redrawn

Commit message: fix trrs top plate
Routing:
- net /KEY17: track 51.3 -> 95.7 mm
- net /TX: track 108.6 -> 103.0 mm
- net /KEY16: track 34.5 -> 39.6 mm
- net GNDR: track 145.0 -> 147.1 mm
Other:
- outline, holes or cut-outs redrawn
