File: pcbs/curcur40/right/curcur40-right.kicad_sch (KiCad schematic)
At the start: 77 parts

Commit message: fix name
Other:
- company: foostan -> curcur40
Changed lines of the file:
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@@
     (date "2023-10-07")
     (rev "1.0.0")
-    (company "foostan")
+    (company "curcur40")
   )
   (junction (at 27.94 184.15) (diameter 0) (color 0 0 0 0)
