File: pcbs/curcur40/right/curcur40-right.kicad_sch (KiCad schematic)
At the start: 77 parts

Commit message: fix
Parts:
- rU4: footprint Package_SO:SOIC-8_5.23x5.23mm_P1.27mm -> Package_SO:SOIC-8_5.3x5.3mm_P1.27mm
Changed lines of the file:
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@@
 			)
 		)
-		(property "Footprint" "Package_SO:SOIC-8_5.23x5.23mm_P1.27mm"
+		(property "Footprint" "Package_SO:SOIC-8_5.3x5.3mm_P1.27mm"
 			(at 228.6 55.88 0)
 			(hide yes)

Commit message: fix pcb
Parts:
- removed rJ3: PMW3360_Conn, kbd_local:PinHeader_1x06_P2.54mm_Vertical, symbol Connector_Generic:Conn_01x06
- added C1: 4.7uF/10V, Capacitor_SMD:C_0603_1608Metric_Pad1.08x0.95mm_HandSolder, symbol Device:C_Small
- added C2: 100nF, Capacitor_SMD:C_0603_1608Metric_Pad1.08x0.95mm_HandSolder, symbol Device:C_Small
- added C3, C4: 1uF, Capacitor_SMD:C_0603_1608Metric_Pad1.08x0.95mm_HandSolder, symbol Device:C_Small
- added C5: 22nF, Capacitor_SMD:C_0603_1608Metric_Pad1.08x0.95mm_HandSolder, symbol Device:C_Small
- added JP1: SolderJumper_3_Open, Jumper:SolderJumper-3_P1.3mm_Open_RoundedPad1.0x1.5mm_NumberLabels, symbol Jumper:SolderJumper_3_Open
- added R1, R2: 10k, Resistor_SMD:R_0603_1608Metric_Pad0.98x0.95mm_HandSolder, symbol Device:R
- added R3: 39R, Resistor_SMD:R_0603_1608Metric_Pad0.98x0.95mm_HandSolder, symbol Device:R
- added R4: 28k, Resistor_SMD:R_0603_1608Metric_Pad0.98x0.95mm_HandSolder, symbol Device:R
- added U1: PMW3360, kbd_local:PMW3360DM-T2QU_16Pin, symbol PMW3360_PCB:PMW3360DM-T2QU
- added U2: TLV74318PDBVR, Package_TO_SOT_SMD:SOT-23-5, symbol PMW3360_PCB:TLV74318PDBVR
Connections:
- net +3V3R: now also C3.1, JP1.1 (A), U2.1 (IN), U2.3 (EN)
- net GNDR: now also C1.2, C2.2, C3.2, C4.2, C5.2, U1.8 (GND), U2.2 (GND)
- net MISO: now also R2.2, U1.12 (MISO)
- net MOSI: now also U1.11 (MOSI)
- net NCS: now also U1.13 (~{CS})
- net SCLK: now also U1.10 (SCLK)
- new net: R3.2, U1.15 (LED_P)
- new net: C1.1, C2.1, U1.3 (VDDPIX)
- new net: C5.1, R4.2, U2.4 (NC)
- new net +1V8_PMW: C4.1, JP1.3 (B), R3.1, R4.1, U1.4 (VDD), U2.5 (OUT)
- new net MOTION: U1.9 (MOTION)
- new net RESET: R1.2, U1.7 (~{RESET})
- new net V_{IO}: JP1.2 (C), R1.1, R2.1, U1.5 (VDDIO)
