File: pcbs/curcur40/left/curcur40-left.kicad_sch (KiCad schematic)
At the start: 79 parts, among them J1 TYPE-C-31-M-13C, J2 TRS, J4 Conn_01x03, SW1 SW_Push, SW10 SW_Push, SW11 SW_Push, SW12 SW_Push, SW13 SW_Push, SW14 SW_Push, SW15 SW_Push, SW16 SW_Push, SW17 SW_Push, SW18 SW_Push, SW2 SW_Push, SW3 SW_Push, SW4 SW_Push, SW5 SW_Push, SW6 SW_Push, SW7 SW_Push, SW8 SW_Push, SW9 SW_Push, U1 RP2040, U2 NCP1117LPST33T3G, U3 TPD4E05U06DQAR, U4 W25Q128JVSIQ, Y1 12MHz 18pF

Commit message: fix name
Other:
- company: foostan -> curcur40
Changed lines of the file:
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@@
     (date "2023-10-07")
     (rev "1.0.0")
-    (company "foostan")
+    (company "curcur40")
   )
   (junction (at 215.9 208.28) (diameter 0) (color 0 0 0 0)
