File: pcbs/curcur40/left/curcur40-left.kicad_pcb (KiCad board)
At the start: 2 copper layers, 124.3 x 91.8 mm, 80 parts, among them J1 TYPE-C-31-M-13C, J2 TRS, J4 Conn_01x03, SW1 SW_Push, SW10 SW_Push, SW11 SW_Push, SW12 SW_Push, SW13 SW_Push, SW14 SW_Push, SW15 SW_Push, SW16 SW_Push, SW17 SW_Push, SW18 SW_Push, SW2 SW_Push, SW3 SW_Push, SW4 SW_Push, SW5 SW_Push, SW6 SW_Push, SW7 SW_Push, SW8 SW_Push, SW9 SW_Push, U1 RP2040, U2 NCP1117LPST33T3G, U3 TPD4E05U06DQAR, U4 W25Q128JVSIQ, Y1 12MHz 18pF

Commit message: fix name
Parts:
- removed G***: LOGO, kbd:corne-logo-horizontal
Other:
- board text added: "curcur40"

Commit message: fix error
Routing:
- net /KEY16: track 58.8 -> 49.6 mm
- net /KEY18: track 84.5 -> 89.8 mm
- net GND: track 202.4 -> 206.6 mm
- net /KEY17: track 64.5 -> 66.1 mm, vias 0 -> 2

Commit message: fix led
Parts:
- moved LED9 1.06 mm to (-71.4, 47.6)
- moved LED8 0.66 mm to (-52.4, 47.6)
Routing:
- net Net-(D1-K): track 555.3 -> 558.8 mm
- net Net-(LED8-DOUT): track 14.7 -> 16.8 mm
- net GND: track 206.6 -> 208.4 mm
- net Net-(LED10-DIN): track 92.1 -> 93.1 mm
Changed lines of the file:
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@@
 	(footprint "kbd_local:YS-SK6812MINI-E"
 		(layer "B.Cu")
-		(at -52.3875 48.3125 180)
+		(at -52.3875 47.65 180)
 		(property "Reference" "LED8"
 			(at 0 1.95 0)
@@
 	(footprint "kbd_local:YS-SK6812MINI-E"
 		(layer "B.Cu")
-		(at -71.4375 48.7125 180)
+		(at -71.4375 47.65 180)
 		(property "Reference" "LED9"
 			(at 0 1.95 0)
@@
 	)
 	(segment
-		(start -68.6375 49.4125)
-		(end -68.3375 49.7125)
-		(width 0.4)
-		(layer "B.Cu")
-		(net "GND")
-	)
-	(segment
 		(start -17.9075 -18.44775)
 		(end -17.9075 -19.0575)
@@
 	)
 	(segment
+		(start -68.338 48.65)
+		(end -68.338 49.712)
+		(width 0.25)
+		(layer "B.Cu")
+		(net "GND")
+	)
+	(segment
+		(start -49.288 48.65)
+		(end -49.288 49.312)
+		(width 0.25)
+		(layer "B.Cu")
+		(net "GND")
+	)
+	(segment
 		(start -76.962498 43.93625)
 		(end -78.112498 43.93625)
@@
 	)
 	(segment
+		(start -49.5875 48.35)
+		(end -49.288 48.65)
+		(width 0.25)
+		(layer "B.Cu")
+		(net "GND")
+	)
+	(segment
 		(start -17.046 -17.70775)
 		(end -17.9075 -18.44775)
@@
 	)
 	(segment
-		(start -49.5875 49.0125)
-		(end -49.2875 49.3125)
-		(width 0.4)
+		(start -68.6375 48.35)
+		(end -68.338 48.65)
+		(width 0.25)
 		(layer "B.Cu")
 		(net "GND")
@@
 	)
 	(segment
-		(start -50.15 46.4625)
-		(end -56 46.4625)
-		(width 0.2)
-		(layer "F.Cu")
-		(net "Net-(D1-K)")
-	)
-	(segment
 		(start -76.8225 19.19125)
 		(end -92.727498 19.19125)
@@
 	)
 	(segment
-		(start -56 46.4625)
-		(end -56 47.6125)
-		(width 0.2)
+		(start -112.3275 -13.63375)
+		(end -113.0625 -14.36875)
+		(width 0.508)
 		(layer "F.Cu")
 		(net "Net-(D1-K)")
 	)
 	(segment
-		(start -112.3275 -13.63375)
-		(end -113.0625 -14.36875)
-		(width 0.508)
+		(start -56.5 45.4)
+		(end -56.5 46.95)
+		(width 0.25)
 		(layer "F.Cu")
 		(net "Net-(D1-K)")
@@
 	)
 	(segment
-		(start -74.35 48.625)
-		(end -73.7375 48.0125)
-		(width 0.2)
-		(layer "F.Cu")
-		(net "Net-(D1-K)")
-	)
-	(segment
 		(start -26.70875 -5.685)
 		(end -26.1575 -5.13375)
@@
 	)
 	(segment
-		(start -74.35 57.7625)
-		(end -74.35 48.625)
-		(width 0.2)
-		(layer "F.Cu")
-		(net "Net-(D1-K)")
-	)
-	(segment
 		(start -36.1375 2.90625)
 		(end -35.6625 2.43125)
@@
 	)
 	(segment
+		(start -50.65 45.4)
+		(end -56.5 45.4)
+		(width 0.25)
+		(layer "F.Cu")
+		(net "Net-(D1-K)")
+	)
+	(segment
 		(start -92.742498 0.23125)
 		(end -93.2875 0.23125)
@@
 	)
 	(segment
+		(start -74.35 46.95)
+		(end -73.7375 46.95)
+		(width 0.25)
+		(layer "F.Cu")
+		(net "Net-(D1-K)")
+	)
+	(segment
 		(start -112.3275 -13.38505)
 		(end -112.3275 -13.388748)
@@
 	)
 	(segment
+		(start -50.15 46.462)
+		(end -50.65 45.4)
+		(width 0.25)
+		(layer "F.Cu")
+		(net "Net-(D1-K)")
+	)
+	(segment
 		(start -55.1575 -18.67375)
 		(end -54.6625 -19.16875)
@@
 	)
 	(segment
+		(start -74.35 57.763)
+		(end -74.35 46.95)
+		(width 0.25)
+		(layer "F.Cu")
+		(net "Net-(D1-K)")
+	)
+	(segment
 		(start -93.358798 19.76995)
 		(end -93.937498 19.19125)
@@
 	)
 	(via
+		(at -56.5 46.95)
+		(size 0.6)
+		(drill 0.3)
+		(layers "F.Cu" "B.Cu")
+		(net "Net-(D1-K)")
+	)
+	(via
 		(at -112.3375 6.46875)
 		(size 0.6)
@@
 	)
 	(via
-		(at -73.7375 48.0125)
-		(size 0.5)
+		(at -73.7375 46.95)
+		(size 0.6)
 		(drill 0.3)
 		(layers "F.Cu" "B.Cu")
@@
 	)
 	(via
-		(at -56 47.6125)
-		(size 0.5)
-		(drill 0.3)
-		(layers "F.Cu" "B.Cu")
-		(net "Net-(D1-K)")
-	)
-	(via
 		(at -23.5 40.135)
 		(size 0.5)
@@
 	)
 	(segment
-		(start -56 47.6125)
-		(end -55.1875 47.6125)
-		(width 0.25)
-		(layer "B.Cu")
-		(net "Net-(D1-K)")
-	)
-	(segment
 		(start -23.0825 -5.05875)
 		(end -23.55875 -4.5825)
@@
 	)
 	(segment
+		(start -56.5 46.95)
+		(end -55.1875 46.95)
+		(width 0.25)
+		(layer "B.Cu")
+		(net "Net-(D1-K)")
+	)
+	(segment
 		(start -17.0875 43)
 		(end -17.0875 46.95)
@@
 	)
 	(segment
-		(start -61 49.6125)
-		(end -67.037499 49.6125)
-		(width 0.2)
+		(start -67 49.8)
+		(end -68.6375 48.1625)
+		(width 0.25)
 		(layer "F.Cu")
 		(net "Net-(LED8-DOUT)")
 	)
 	(segment
-		(start -67.037499 49.6125)
-		(end -68.6375 48.0125)
-		(width 0.2)
+		(start -68.6375 48.1625)
+		(end -68.6375 46.95)
+		(width 0.25)
+		(layer "F.Cu")
+		(net "Net-(LED8-DOUT)")
+	)
+	(segment
+		(start -57.5 48.35)
+		(end -57.5 49.8)
+		(width 0.25)
+		(layer "F.Cu")
+		(net "Net-(LED8-DOUT)")
+	)
+	(segment
+		(start -57.5 49.8)
+		(end -67 49.8)
+		(width 0.25)
 		(layer "F.Cu")
 		(net "Net-(LED8-DOUT)")
 	)
 	(via
-		(at -68.6375 48.0125)
-		(size 0.5)
+		(at -68.6375 46.95)
+		(size 0.6)
 		(drill 0.3)
 		(layers "F.Cu" "B.Cu")
@@
 	)
 	(via
-		(at -61 49.6125)
-		(size 0.5)
+		(at -57.5 48.35)
+		(size 0.6)
 		(drill 0.3)
 		(layers "F.Cu" "B.Cu")
@@
 	)
 	(segment
-		(start -61 49.0125)
-		(end -61 49.6125)
-		(width 0.2)
-		(layer "B.Cu")
-		(net "Net-(LED8-DOUT)")
-	)
-	(segment
-		(start -55.1875 49.0125)
-		(end -61 49.0125)
-		(width 0.2)
+		(start -55.1875 48.35)
+		(end -57.5 48.35)
+		(width 0.25)
 		(layer "B.Cu")
 		(net "Net-(LED8-DOUT)")
@@
 	)
 	(segment
+		(start -48.924 46.95)
+		(end -49.5875 46.95)
+		(width 0.25)
+		(layer "B.Cu")
+		(net "Net-(LED7-DOUT)")
+	)
+	(segment
 		(start -55.18375 22.15625)
 		(end -55.1725 22.145)
@@
 	)
 	(segment
-		(start -48.4325 46.4575)
-		(end -49.5875 47.6125)
+		(start -48.4325 39.7762)
+		(end -48.4325 46.4575)
 		(width 0.2)
 		(layer "B.Cu")
@@
 	)
 	(segment
-		(start -48.4325 39.7762)
-		(end -48.4325 46.4575)
-		(width 0.2)
+		(start -48.432 46.458)
+		(end -48.924 46.95)
+		(width 0.25)
 		(layer "B.Cu")
 		(net "Net-(LED7-DOUT)")
@@
 	)
 	(segment
-		(start -74.3 62.0025)
-		(end -74.3 49.4125)
-		(width 0.2)
+		(start -68.6375 18.375)
+		(end -68.6625 18.375)
+		(width 0.2032)
 		(layer "B.Cu")
 		(net "Net-(LED10-DIN)")
 	)
 	(segment
-		(start -74.3 49.4125)
-		(end -73.7375 49.4125)
+		(start -74.3 62.002)
+		(end -74.3 48.35)
 		(width 0.2)
 		(layer "B.Cu")
@@
 	)
 	(segment
-		(start -64.599999 62.0025)
-		(end -74.3 62.0025)
+		(start -60.5 40.55)
+		(end -60.5 48.3125)
 		(width 0.2)
 		(layer "B.Cu")
@@
 	)
 	(segment
-		(start -68.6375 18.375)
-		(end -68.6625 18.375)
-		(width 0.2032)
+		(start -64.599999 62.002)
+		(end -74.3 62.002)
+		(width 0.2)
 		(layer "B.Cu")
 		(net "Net-(LED10-DIN)")
 	)
 	(segment
-		(start -60.5 40.55)
-		(end -60.5 48.3125)
+		(start -74.3 48.35)
+		(end -73.7375 48.35)
 		(width 0.2)
 		(layer "B.Cu")
