File: plates/curcur40/pcb/plate-bottom-right.kicad_pcb (KiCad board)
At the start: 2 copper layers, 125.1 x 92.6 mm, 0 parts

Commit message: mv trackball hole
Other:
- outline, holes or cut-outs redrawn
Changed lines of the file:
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@@
 	)
 	(gr_circle
-		(center 4.725 41.0875)
-		(end 5.825 41.0875)
+		(center -2.474999 41.0875)
+		(end -1.374999 41.0875)
 		(stroke
 			(width 0.15)
@@
 	)
 	(gr_circle
-		(center 4.725 63.6875)
-		(end 5.825 63.6875)
+		(center -2.474999 63.6875)
+		(end -1.374999 63.6875)
 		(stroke
 			(width 0.15)
@@
 	)
 	(gr_circle
-		(center 14.325 41.0875)
-		(end 15.424999 41.0875)
+		(center 21.525 41.0875)
+		(end 22.625 41.0875)
 		(stroke
 			(width 0.15)
@@
 	)
 	(gr_circle
-		(center 14.325 63.6875)
-		(end 15.424999 63.6875)
+		(center 21.525 63.6875)
+		(end 22.625 63.6875)
 		(stroke
 			(width 0.15)
