File: pcbs/left/curcur40-left.kicad_pcb (KiCad board)
At the start: 2 copper layers, 124.3 x 91.8 mm, 79 parts, among them J1 TYPE-C-31-M-13C, J2 TRS, J4 Conn_01x03, SW1 SW_Push, SW10 SW_Push, SW11 SW_Push, SW12 SW_Push, SW13 SW_Push, SW14 SW_Push, SW15 SW_Push, SW16 SW_Push, SW17 SW_Push, SW18 SW_Push, SW2 SW_Push, SW3 SW_Push, SW4 SW_Push, SW5 SW_Push, SW6 SW_Push, SW7 SW_Push, SW8 SW_Push, SW9 SW_Push, U1 RP2040, U2 NCP1117LPST33T3G, U3 TPD4E05U06DQAR, U4 W25Q128JVSIQ, Y1 12MHz 18pF

Commit message: fix(pcb): update spacer holes to 3.25mm, shift SMDSW1/2, remove 0.4mm NPTH hole, and sync U1/CKW12 attributes
Parts:
- moved SMDSW1 0.77 mm to (-94.2, 37.3)
- moved SMDSW2 0.52 mm to (-90.6, 37.3)
Routing:
- net GND: track 210.0 -> 210.6 mm
Other:
- outline, holes or cut-outs redrawn

Commit message: feat(pcb): separate pmw3360 sensor PCB with JST SH 6-pin connector and add symmetric thumb mounting holes L5/R5
Other:
- outline, holes or cut-outs redrawn
Changed lines of the file:
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@@
 	)
 	(gr_circle
-		(center -21.525 63.6875)
-		(end -19.9 63.6875)
+		(center -33.3375 64.3)
+		(end -31.7125 64.3)
 		(stroke
 			(width 0.1)

Commit message: feat(pcb,plates): face-to-face JST SH orientation, move TRRS jack north, and refine mounting holes
Parts:
- moved J2 5.00 mm to (5.26, 29.6)
Routing:
- net +5V: track 129.8 -> 139.7 mm
- net /TX: track 141.1 -> 149.3 mm
Other:
- outline, holes or cut-outs redrawn
Changed lines of the file:
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@@
 	(footprint "kbd:Jack_PJ-398A-5A_PJ-399B-6A"
 		(layer "B.Cu")
-		(at 5.2575 34.64625 90)
+		(at 5.2575 29.6463 90)
 		(tags "usb usb-c 2.0 pd")
 		(property "Reference" "J2"
@@
 	)
 	(gr_circle
-		(center -109.5375 -20)
-		(end -107.9125 -20)
+		(center -101 -20)
+		(end -99.375 -20)
 		(stroke
 			(width 0.1)
@@
 	)
 	(gr_circle
-		(center -33.3375 64.3)
-		(end -31.7125 64.3)
+		(center -62 64.599999)
+		(end -60.375 64.599999)
 		(stroke
 			(width 0.1)
@@
 	)
 	(gr_line
-		(start -7.7425 31.5)
-		(end -7.7425 37.8)
+		(start -7.7425 26.5)
+		(end -7.7425 32.799999)
 		(stroke
-			(width 0.1)
+			(width 0.15)
 			(type default)
 		)
@@
 	)
 	(gr_line
-		(start -7.7425 37.8)
-		(end 5.2625 37.8)
+		(start -7.7425 32.799999)
+		(end 5.2625 32.799999)
 		(stroke
-			(width 0.1)
+			(width 0.15)
 			(type default)
 		)
@@
 	)
 	(gr_circle
-		(center 0 25)
-		(end 1.625 25)
+		(center 0 20)
+		(end 1.625 20)
 		(stroke
 			(width 0.1)
@@
 	(gr_line
 		(start 5.2625 -23.3125)
-		(end 5.2625 31.5)
+		(end 5.2625 26.5)
 		(stroke
-			(width 0.1)
+			(width 0.15)
 			(type default)
 		)
@@
 	)
 	(gr_line
-		(start 5.2625 31.5)
-		(end -7.7425 31.5)
+		(start 5.2625 26.5)
+		(end -7.7425 26.5)
 		(stroke
-			(width 0.1)
+			(width 0.15)
 			(type default)
 		)
@@
 	)
 	(gr_line
-		(start 5.2625 37.8)
+		(start 5.2625 32.799999)
 		(end 5.2625 66.5)
 		(stroke
-			(width 0.1)
+			(width 0.15)
 			(type default)
 		)
@@
 	)
 	(segment
+		(start -8.5 38.62)
+		(end -8.5 33.5463)
+		(width 0.4)
+		(layer "B.Cu")
+		(net "+5V")
+	)
+	(segment
 		(start -39.24256 41.233382)
 		(end -39.919068 41.233382)
@@
 	)
 	(segment
+		(start -8.5 25.7462)
+		(end -6.5425 25.7462)
+		(width 0.4)
+		(layer "B.Cu")
+		(net "+5V")
+	)
+	(segment
+		(start -8.5 33.5463)
+		(end -6.5425 33.5463)
+		(width 0.4)
+		(layer "B.Cu")
+		(net "+5V")
+	)
+	(segment
 		(start -25.0625 -5.735)
 		(end -24.3425 -5.735)
@@
 	)
 	(segment
-		(start -8.5 38.62)
-		(end -6.5425 38.54625)
-		(width 0.4)
-		(layer "B.Cu")
-		(net "+5V")
-	)
-	(segment
 		(start -8.5 30.596)
-		(end -6.5425 30.74625)
+		(end -8.5 25.7462)
 		(width 0.4)
 		(layer "B.Cu")
@@
 	)
 	(segment
-		(start -0.7425 29)
-		(end -10 29)
+		(start -9.6 40)
+		(end -6.1 40)
 		(width 0.25)
 		(layer "B.Cu")
@@
 	)
 	(segment
-		(start -67.29 42.08)
-		(end -67.29 43.3)
-		(width 0.2)
+		(start -0.7425 24.5)
+		(end -9.6 24.5)
+		(width 0.25)
 		(layer "B.Cu")
 		(net "/TX")
 	)
 	(segment
-		(start -0.7425 40)
-		(end -0.7425 38.54625)
-		(width 0.25)
+		(start -67.29 42.08)
+		(end -67.29 43.3)
+		(width 0.2)
 		(layer "B.Cu")
 		(net "/TX")
@@
 	)
 	(segment
-		(start -6.1 40)
-		(end -0.7425 40)
-		(width 0.25)
-		(layer "B.Cu")
-		(net "/TX")
-	)
-	(segment
 		(start -19.4325 60.8)
 		(end -18.65 61.5825)
@@
 	)
 	(segment
-		(start -10 29)
-		(end -10 40)
-		(width 0.25)
+		(start -64 61.5825)
+		(end -24.4 61.5825)
+		(width 0.2)
 		(layer "B.Cu")
 		(net "/TX")
 	)
 	(segment
-		(start -0.7425 30.74625)
-		(end -0.7425 29)
+		(start -0.7425 33.5463)
+		(end -0.7425 40)
 		(width 0.25)
 		(layer "B.Cu")
@@
 	)
 	(segment
-		(start -64 61.5825)
-		(end -24.4 61.5825)
+		(start -64 43.3)
+		(end -64 61.5825)
 		(width 0.2)
 		(layer "B.Cu")
@@
 	)
 	(segment
-		(start -10 40)
+		(start -18.65 61.5825)
+		(end -6.1 61.5825)
+		(width 0.2)
+		(layer "B.Cu")
+		(net "/TX")
+	)
+	(segment
+		(start -0.7425 40)
 		(end -6.1 40)
 		(width 0.25)
@@
 	)
 	(segment
-		(start -64 43.3)
-		(end -64 61.5825)
-		(width 0.2)
+		(start -0.7425 25.7462)
+		(end -0.7425 24.5)
+		(width 0.25)
 		(layer "B.Cu")
 		(net "/TX")
 	)
 	(segment
-		(start -18.65 61.5825)
-		(end -6.1 61.5825)
-		(width 0.2)
+		(start -9.6 24.5)
+		(end -9.6 40)
+		(width 0.25)
 		(layer "B.Cu")
 		(net "/TX")
