File: pcbs/right/curcur40-right.kicad_pcb (KiCad board)
At the start: 2 copper layers, 124.3 x 91.8 mm, 88 parts, among them U1 PMW3360DM-T2QU, U2 TLV74318PDBVR

Commit message: feat(pcb): separate pmw3360 sensor PCB with JST SH 6-pin connector and add symmetric thumb mounting holes L5/R5
Parts:
- removed C1: 4.7uF/10V, Capacitor_SMD:C_0603_1608Metric_Pad1.08x0.95mm_HandSolder
- removed C2: 100nF, Capacitor_SMD:C_0603_1608Metric_Pad1.08x0.95mm_HandSolder
- removed C3, C4: 1uF, Capacitor_SMD:C_0603_1608Metric_Pad1.08x0.95mm_HandSolder
- removed C5: 22nF, Capacitor_SMD:C_0603_1608Metric_Pad1.08x0.95mm_HandSolder
- removed JP1: SolderJumper_3_Bridged12, Jumper:SolderJumper-3_P1.3mm_Bridged12_RoundedPad1.0x1.5mm_NumberLabels
- removed R1, R2: 10k, Resistor_SMD:R_0603_1608Metric_Pad0.98x0.95mm_HandSolder
- removed R3: 39R, Resistor_SMD:R_0603_1608Metric_Pad0.98x0.95mm_HandSolder
- removed R4: 28k, Resistor_SMD:R_0603_1608Metric_Pad0.98x0.95mm_HandSolder
- removed U1: PMW3360DM-T2QU, kbd:PMW3360DM-T2QU_16Pin
- removed U2: TLV74318PDBVR, Package_TO_SOT_SMD:SOT-23-5
- added rJ3: SM06B-SRSS-TB, Connector_JST:JST_SH_SM06B-SRSS-TB_1x06-1MP_P1.00mm_Horizontal, B.Cu at (45.0, 63.9)
Routing:
- net GNDR: track 275.8 -> 204.4 mm, vias 60 -> 63
- net /MISO: track 133.9 -> 62.9 mm, vias 4 -> 2
- net +3V3R: track 307.2 -> 240.8 mm, vias 19 -> 14
- net /+1V8_PMW: track 65.1 -> 0.00 mm, vias 2 -> 0
- net Net-(U1-LED_P): track 55.1 -> 0.00 mm, vias 1 -> 0
- net /MOSI: track 99.9 -> 58.3 mm, vias 3 -> 2
- net /SCLK: track 99.3 -> 58.9 mm, vias 3 -> 2
- net /V_{IO}: track 36.5 -> 0.00 mm, vias 1 -> 0
- net /NCS: track 128.9 -> 164.7 mm
- net Net-(U1-VDDPIX): track 30.4 -> 0.00 mm
- net /RESET: track 26.0 -> 0.00 mm, vias 1 -> 0
- net Net-(U2-NC): track 16.3 -> 0.00 mm, vias 2 -> 0
- net /TX: track 100.9 -> 96.8 mm
- net /USB_VBUS_PIN: track 114.8 -> 114.2 mm
Other:
- outline, holes or cut-outs redrawn

Commit message: feat(pcb,plates): face-to-face JST SH orientation, move TRRS jack north, and refine mounting holes
Parts:
- moved rJ2 5.00 mm to (-5.26, 29.6)
- moved rJ3 3.27 mm to (42.0, 62.6), turned to 90 degrees
Routing:
- net /NCS: track 164.7 -> 155.0 mm
- net +5VR: track 123.3 -> 113.8 mm, vias 5 -> 4
- net /TX: track 96.8 -> 101.3 mm
- net /MISO: track 62.9 -> 66.8 mm, vias 2 -> 4
- net +3V3R: track 240.8 -> 238.5 mm, vias 14 -> 16
- net /MOSI: track 58.3 -> 57.0 mm
- net /SCLK: track 58.9 -> 57.8 mm, vias 2 -> 4
- net /KEYEX2: track 97.0 -> 97.8 mm, vias 0 -> 2
- net GNDR: track 204.4 -> 204.1 mm, vias 63 -> 62
Other:
- outline, holes or cut-outs redrawn
