File: pcbs/right/curcur40-right.kicad_pcb (KiCad board)
At the start: 2 copper layers, 124.3 x 91.8 mm, 77 parts

Commit message: feat(pcb): shift rJ3 east to (46.5, 63.0) for rSW1 socket clearance and align N-S pin order with J1
Parts:
- moved rJ3 4.52 mm to (46.5, 63.0)
Connections:
- rJ3 pad 1: +3V3R -> /NCS
- rJ3 pad 2: GNDR -> /MISO
- rJ3 pad 3: /SCLK -> /MOSI
- rJ3 pad 4: /MOSI -> /SCLK
- rJ3 pad 5: /MISO -> GNDR
- rJ3 pad 6: /NCS -> +3V3R
Routing:
- net /NCS: track 155.0 -> 165.5 mm
- net GNDR: track 204.1 -> 213.4 mm
- net +3V3R: track 238.5 -> 229.7 mm, vias 16 -> 14
- net /MISO: track 66.8 -> 59.4 mm, vias 4 -> 2
- net /SCLK: track 57.8 -> 51.9 mm, vias 4 -> 2
- net /MOSI: track 57.0 -> 53.1 mm

Commit message: feat(pcb): replace split TRRS jack with USB-C receptacle and ESD/series protection
Parts:
- added rC17: 100n, Capacitor_SMD:C_0402_1005Metric, B.Cu at (8.80, 26.6)
- added rR10: 27, Resistor_SMD:R_0402_1005Metric, B.Cu at (7.20, 34.8)
- added rU5: TPD4E05U06DQAR, Package_SON:USON-10_2.5x1.0mm_P0.5mm, B.Cu at (4.20, 30.0)
- rJ2: value TRS -> TYPE-C-31-M-13C; footprint kbd:Jack_PJ-398A-5A_PJ-399B-6A -> kbd:USB_C_Receptacle_TYPE-C-31-M-13C
- moved rJ2 1.26 mm to (-4.01, 29.5), turned to 90 degrees
Routing:
- net /TX: track 101.3 -> 76.9 mm, vias 3 -> 2
- net /SPLIT_DP: track 0.00 -> 15.4 mm
- net GNDR: track 213.4 -> 223.9 mm, vias 62 -> 63
- net +5VR: track 113.8 -> 121.3 mm, vias 4 -> 6
Other:
- outline, holes or cut-outs redrawn

Commit message: feat(pcb): integrate sunk inertia wheel cutout and rJ5 connector into curcur40-right and top plate
Parts:
- removed rEXSW1: CKW12, kbd:RotaryEncoder_Switch_CKW12
- added rC18: 100n, Capacitor_SMD:C_0402_1005Metric, B.Cu at (20.1, 34.0)
- added rJ5: SM06B-SRSS-TB, Connector_JST:JST_SH_SM06B-SRSS-TB_1x06-1MP_P1.00mm_Horizontal, B.Cu at (15.8, 32.0)
- added rR11: 4.7k, Resistor_SMD:R_0402_1005Metric, B.Cu at (23.3, 25.0)
- added rR12: 4.7k, Resistor_SMD:R_0402_1005Metric, B.Cu at (23.3, 26.5)
- moved rR2 1.21 mm to (19.4, -16.5)
Connections:
- rU1 pad 36: /RE0A -> /WHEEL_SDA
- rU1 pad 37: /KEYEX1 -> /WHEEL_SCL
- rU1 pad 9: /REB -> /KEYEX1
Routing:
- net /REB: track 127.6 -> 0.00 mm, vias 6 -> 0
- net /RE0A: track 96.3 -> 0.00 mm, vias 1 -> 0
- net /WHEEL_SCL: track 0.00 -> 88.4 mm, vias 0 -> 4
- net /WHEEL_SDA: track 0.00 -> 87.9 mm, vias 0 -> 4
- net GNDR: track 223.9 -> 282.4 mm, vias 63 -> 70
- net +3V3R: track 229.7 -> 273.2 mm, vias 14 -> 18
- net /D-: track 147.5 -> 123.5 mm, vias 6 -> 4
- net Net-(rD1-K): track 469.7 -> 446.8 mm, vias 27 -> 24
- net /D+: track 142.5 -> 120.9 mm
- net /KEYEX1: track 87.3 -> 104.1 mm, vias 2 -> 6
- net Net-(rEXLED2-DIN): track 140.4 -> 128.1 mm, vias 2 -> 4
- net VBUSR: track 29.2 -> 17.9 mm
- net Net-(rJ1-CC2): track 18.2 -> 6.95 mm
- net Net-(rJ1-CC1): track 18.6 -> 8.54 mm
- net /KEYEX2: track 97.8 -> 97.1 mm
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Other:
- outline, holes or cut-outs redrawn
