File: pcbs/pmw3360/curcur40-pmw3360.kicad_sch (KiCad schematic)
At the start: 13 parts, among them J1 SM06B-SRSS-TB, U1 PMW3360DM-T2QU, U2 TLV74318PDBVR

Commit message: fix(bom,pcb): update JST SH 6-pin connector LCSC part number from C160404 to C160405
Parts:
- J1: LCSC C160404 -> C160405
Changed lines of the file:
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@@
 			)
 		)
-		(property "LCSC" "C160404"
+		(property "LCSC" "C160405"
 			(at 279.4 101.6 0)
 			(effects
