File: pcbs/inertia-wheel-eval/curcur40-wheel-eval.kicad_sch (KiCad schematic)
At the start: 7 parts, among them J1 SM06B-SRSS-TB, J2 AS5600_Wires, SW1 Kailh_Silent_6.2x6.2, U1 Waveshare_RP2040-Zero

Commit message: feat(pcb): integrate sunk inertia wheel cutout and rJ5 connector into curcur40-right and top plate
Connections:
- net GND: now also J1.6 (Pin_6)
- no-connect marks 19 -> 18
Changed lines of the file:
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@@
 	(wire (pts (xy 175.26 106.68) (xy 185.42 106.68)) (stroke (width 0) (type default)))
 	(label "SW_MID" (at 175.26 106.68 0) (effects (font (size 1.27 1.27)) (justify left bottom)))
-	(no_connect (at 185.42 109.22))
 	(symbol
 		(lib_id "power:GND")
+		(at 180.34 111.76 0)
+		(unit 1)
+		(exclude_from_sim no)
+		(in_bom no)
+		(on_board no)
+		(dnp no)
+		(property "Reference" "#PWR21" (at 180.34 107.95 0) (effects (font (size 1.27 1.27))))
+		(property "Value" "GND" (at 180.34 115.57 0) (effects (font (size 1.27 1.27))))
+		(property "Footprint" "" (at 180.34 111.76 0) (hide yes) (effects (font (size 1.27 1.27))))
+		(property "Datasheet" "" (at 180.34 111.76 0) (hide yes) (effects (font (size 1.27 1.27))))
+		(instances (project "curcur40-wheel-eval" (path "/e59eea65-32d5-5ecb-89d9-210ef6b13dc1" (reference "#PWR21") (unit 1))))
+	)
+	(wire (pts (xy 180.34 111.76) (xy 180.34 109.22)) (stroke (width 0) (type default)))
+	(wire (pts (xy 180.34 109.22) (xy 185.42 109.22)) (stroke (width 0) (type default)))
+	(symbol
+		(lib_id "power:GND")
